File: First_PCB/First_PCB.kicad_sch (KiCad schematic)
At the start: 3 parts, among them J1 Conn_01x02

Commit message: .
Parts:
- added D2: SK6812MINI, LED_SMD:LED_SK6812MINI_PLCC4_3.5x3.5mm_P1.75mm, symbol LED:SK6812MINI
- added U1: ESP32-PICO-D4, Package_DFN_QFN:QFN-48-1EP_7x7mm_P0.5mm_EP5.3x5.3mm, symbol RF_Module:ESP32-PICO-D4
- J1: footprint (none) -> Connector_PinSocket_2.54mm:PinSocket_1x02_P2.54mm_Vertical
- R1: footprint (none) -> Resistor_SMD:R_0603_1608Metric
Connections:
- net at J1.1 (Pin_1), R1.1: now also D2.4 (VDD), U1.1 (VDDA), U1.19 (VDD3P3_RTC), U1.3 (VDDA3P3), U1.37 (VDD3P3_CPU), U1.4 (VDDA3P3), U1.43 (VDDA), U1.46 (VDDA)
- net GND: now reaches D1.1 (K), J1.2 (Pin_2)
- net GND: now also D2.2 (VSS), U1.49 (GND)
- new net: D2.3 (DIN), U1.22 (IO2)
Changed lines of the file:
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@@
 (kicad_sch (version 20230121) (generator eeschema)
   (paper "A4")
+  (junction (at 161.29 104.14) (diameter 0) (color 0 0 0 0)
+  )
+  (junction (at 83.82 86.36) (diameter 0) (color 0 0 0 0)
+  )
+  (junction (at 88.9 86.36) (diameter 0) (color 0 0 0 0)
+  )
+  (junction (at 86.36 86.36) (diameter 0) (color 0 0 0 0)
+  )
+  (junction (at 171.45 81.28) (diameter 0) (color 0 0 0 0)
+  )
+  (junction (at 91.44 86.36) (diameter 0) (color 0 0 0 0)
+  )
+  (junction (at 172.72 78.74) (diameter 0) (color 0 0 0 0)
+  )
+  (junction (at 171.45 104.14) (diameter 0) (color 0 0 0 0)
+  )
+  (wire (pts (xy 83.82 86.36) (xy 86.36 86.36))
+    (stroke (width 0) (type default))
+  )
+  (wire (pts (xy 172.72 78.74) (xy 172.72 63.5))
+    (stroke (width 0) (type default))
+  )
+  (wire (pts (xy 161.29 173.99) (xy 161.29 104.14))
+    (stroke (width 0) (type default))
+  )
   (wire (pts (xy 168.91 78.74) (xy 172.72 78.74))
     (stroke (width 0) (type default))
   )
-  (wire (pts (xy 151.13 81.28) (xy 172.72 81.28))
+  (wire (pts (xy 171.45 104.14) (xy 175.26 104.14))
+    (stroke (width 0) (type default))
+  )
+  (wire (pts (xy 83.82 63.5) (xy 83.82 86.36))
+    (stroke (width 0) (type default))
+  )
+  (wire (pts (xy 153.67 107.95) (xy 153.67 96.52))
+    (stroke (width 0) (type default))
+  )
+  (wire (pts (xy 86.36 86.36) (xy 86.36 92.71))
+    (stroke (width 0) (type default))
+  )
+  (wire (pts (xy 151.13 81.28) (xy 171.45 81.28))
+    (stroke (width 0) (type default))
+  )
+  (wire (pts (xy 171.45 81.28) (xy 171.45 104.14))
+    (stroke (width 0) (type default))
+  )
+  (wire (pts (xy 161.29 86.36) (xy 161.29 88.9))
+    (stroke (width 0) (type default))
+  )
+  (wire (pts (xy 172.72 63.5) (xy 83.82 63.5))
     (stroke (width 0) (type default))
   )
@@
     (stroke (width 0) (type default))
   )
+  (wire (pts (xy 86.36 86.36) (xy 88.9 86.36))
+    (stroke (width 0) (type default))
+  )
+  (wire (pts (xy 175.26 104.14) (xy 175.26 105.41))
+    (stroke (width 0) (type default))
+  )
+  (wire (pts (xy 91.44 86.36) (xy 161.29 86.36))
+    (stroke (width 0) (type default))
+  )
+  (wire (pts (xy 161.29 104.14) (xy 171.45 104.14))
+    (stroke (width 0) (type default))
+  )
+  (wire (pts (xy 83.82 86.36) (xy 83.82 92.71))
+    (stroke (width 0) (type default))
+  )
+  (wire (pts (xy 88.9 86.36) (xy 88.9 92.71))
+    (stroke (width 0) (type default))
+  )
+  (wire (pts (xy 88.9 86.36) (xy 91.44 86.36))
+    (stroke (width 0) (type default))
+  )
+  (wire (pts (xy 171.45 81.28) (xy 172.72 81.28))
+    (stroke (width 0) (type default))
+  )
+  (wire (pts (xy 88.9 173.99) (xy 161.29 173.99))
+    (stroke (width 0) (type default))
+  )
+  (wire (pts (xy 153.67 107.95) (xy 109.22 107.95))
+    (stroke (width 0) (type default))
+  )
   (wire (pts (xy 158.75 78.74) (xy 161.29 78.74))
     (stroke (width 0) (type default))
   )
+  (wire (pts (xy 91.44 86.36) (xy 91.44 92.71))
+    (stroke (width 0) (type default))
+  )
   (symbol (lib_id "Device:R") (at 165.1 78.74 270) (unit 1)
     (in_bom yes) (on_board yes) (dnp no) (fields_autoplaced)
@@
       (effects (font (size 1.27 1.27)))
     )
-    (property "Footprint" "" (at 165.1 76.962 90)
+    (property "Footprint" "Resistor_SMD:R_0603_1608Metric" (at 165.1 76.962 90)
       (effects (font (size 1.27 1.27)) hide)
     )
@@
       (effects (font (size 1.27 1.27)) (justify left))
     )
-    (property "Footprint" "" (at 177.8 78.74 0)
+    (property "Footprint" "Connector_PinSocket_2.54mm:PinSocket_1x02_P2.54mm_Vertical" (at 177.8 78.74 0)
       (effects (font (size 1.27 1.27)) hide)
     )
@@
         )
       )
+    )
+  )
+  (symbol (lib_id "LED:SK6812MINI") (at 161.29 96.52 0) (unit 1)
+    (in_bom yes) (on_board yes) (dnp no) (fields_autoplaced)
+    (property "Reference" "D2" (at 173.99 92.8721 0)
+      (effects (font (size 1.27 1.27)))
+    )
+    (property "Value" "SK6812MINI" (at 173.99 95.4121 0)
+      (effects (font (size 1.27 1.27)))
+    )
+    (property "Footprint" "LED_SMD:LED_SK6812MINI_PLCC4_3.5x3.5mm_P1.75mm" (at 162.56 104.14 0)
+      (effects (font (size 1.27 1.27)) (justify left top) hide)
+    )
+    (property "Datasheet" "https://cdn-shop.adafruit.com/product-files/2686/SK6812MINI_REV.01-1-2.pdf" (at 163.83 106.045 0)
+      (effects (font (size 1.27 1.27)) (justify left top) hide)
+    )
+    (pin "1")
+    (pin "2")
+    (pin "3")
+    (pin "4")
+    (instances
+      (project "First_PCB"
+        (path "/40b759d2-5493-4b00-830e-f3c37aad9b46"
+          (reference "D2") (unit 1)
+        )
+      )
+    )
+  )
+  (symbol (lib_id "power:GND") (at 175.26 105.41 0) (unit 1)
+    (in_bom yes) (on_board yes) (dnp no) (fields_autoplaced)
+    (property "Reference" "#PWR03" (at 175.26 111.76 0)
+      (effects (font (size 1.27 1.27)) hide)
+    )
+    (property "Value" "GND" (at 175.26 110.49 0)
+      (effects (font (size 1.27 1.27)))
+    )
+    (property "Footprint" "" (at 175.26 105.41 0)
+      (effects (font (size 1.27 1.27)) hide)
+    )
+    (property "Datasheet" "" (at 175.26 105.41 0)
+      (effects (font (size 1.27 1.27)) hide)
+    )
+    (pin "1")
+    (instances
+      (project "First_PCB"
+        (path "/40b759d2-5493-4b00-830e-f3c37aad9b46"
+          (reference "#PWR03") (unit 1)
+        )
+      )
+    )
+  )
+  (symbol (lib_id "RF_Module:ESP32-PICO-D4") (at 88.9 133.35 0) (unit 1)
+    (in_bom yes) (on_board yes) (dnp no) (fields_autoplaced)
+    (property "Reference" "U1" (at 91.0941 173.99 0)
+      (effects (font (size 1.27 1.27)) (justify left))
+    )
+    (property "Value" "ESP32-PICO-D4" (at 91.0941 176.53 0)
+      (effects (font (size 1.27 1.27)) (justify left))
+    )
+    (property "Footprint" "Package_DFN_QFN:QFN-48-1EP_7x7mm_P0.5mm_EP5.3x5.3mm" (at 88.9 176.53 0)
+      (effects (font (size 1.27 1.27)) hide)
+    )
+    (property "Datasheet" "https://www.espressif.com/sites/default/files/documentation/esp32-pico-d4_datasheet_en.pdf" (at 95.25 158.75 0)
+      (effects (font (size 1.27 1.27)) hide)
+    )
+    (pin "1")
+    (pin "10")
+    (pin "11")
+    (pin "12")
+    (pin "13")
+    (pin "14")
+    (pin "15")
+    (pin "16")
+    (pin "17")
+    (pin "18")
+    (pin "19")
+    (pin "2")
+    (pin "20")
+    (pin "21")
+    (pin "22")
+    (pin "23")
+    (pin "24")
+    (pin "25")
+    (pin "26")
+    (pin "27")
+    (pin "28")
+    (pin "29")
+    (pin "3")
+    (pin "30")
+    (pin "31")
+    (pin "32")
+    (pin "33")
+    (pin "34")
+    (pin "35")
+    (pin "36")
+    (pin "37")
+    (pin "38")
+    (pin "39")
+    (pin "4")
+    (pin "40")
+    (pin "41")
+    (pin "42")
+    (pin "43")
+    (pin "44")
+    (pin "45")
+    (pin "46")
+    (pin "47")
+    (pin "48")
+    (pin "49")
+    (pin "5")
+    (pin "6")
+    (pin "7")
+    (pin "8")
+    (pin "9")
+    (instances
+      (project "First_PCB"
+        (path "/40b759d2-5493-4b00-830e-f3c37aad9b46"
+          (reference "U1") (unit 1)
+        )
+      )
