File: ESP32_Solenoid/ESP32_Solenoid.kicad_sch (KiCad schematic)
At the start: 21 parts, among them J1 PowerInput, J2 PhotoMicroSensor, J3 CAN_Socket, J4 Solenoid, Q1 IRLZ44N, Q2 BSS138, U1 DRV8313PWP, U2 Xiao_ESP32S3, U3 SN65HVD230DR

Commit message: .
Parts:
- added U4: MP1584EN, MP1584EN:SOIC127P600X170-9N, symbol MP1584EN:MP1584EN
Connections:
- net +24V: now also U4.7 (VIN)
- net GND: now also U4.5 (GND), U4.9 (GND)
Other:
- moved on the sheet: J4, U1
